File: DBCon.brd (EAGLE design)
At the start: 100 x 87.6 mm, 100 parts, among them M1 1_PIN, M10 1_PIN, M11 1_PIN, M12 1_PIN, M13 1_PIN, M14 1_PIN, M2 1_PIN, M3 1_PIN, M4 1_PIN, M5 1_PIN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

Commit message: Freed up analog pin
Connections:
- net CLK: now also B1.13; no longer B1.20
Routing:
- net CLK: track 12.5 -> 29.6 mm, vias 0 -> 2
Changed lines of the file:
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@@
 <signal name="CLK">
 <contactref element="SN74HC163D_1" pad="2"/>
-<contactref element="B1" pad="20"/>
-<wire x1="81.28" y1="12.7" x2="79.375" y2="13.335" width="0.4064" layer="1"/>
-<wire x1="79.375" y1="13.335" x2="68.84" y2="13.335" width="0.4064" layer="1"/>
+<contactref element="B1" pad="13"/>
+<wire x1="68.84" y1="13.335" x2="72.39" y2="13.335" width="0.4064" layer="1"/>
+<wire x1="72.39" y1="13.335" x2="72.39" y2="16.51" width="0.4064" layer="1"/>
+<via x="72.39" y="16.51" extent="1-16" drill="0.6" shape="square"/>
+<wire x1="72.39" y1="16.51" x2="72.39" y2="30.48" width="0.4064" layer="16"/>
+<via x="72.39" y="30.48" extent="1-16" drill="0.6" shape="square"/>
+<wire x1="72.39" y1="30.48" x2="81.28" y2="30.48" width="0.4064" layer="1"/>
 </signal>
 <signal name="A">
